File: eagle/kiev_nrf2401_reva.sch (EAGLE design)
At the start: 5 parts

Commit message: Making design open
Parts:
- removed U$1: MRF24J40MA, eurosource_mrf24j40ma:MRF24J40MA
- added SV1: JP2, con-lstb:MA04-2
- renumbered C2 to C3
Connections:
- removed net CS_MRF24J40MA: JP1.3, R1.1, U$1./CS
- removed net INT0: JP1.18, U$1.INT
- removed net N$25: JP1.13
- removed net RESET: JP1.14, U$1./RESET
- removed net SCK1: JP1.5, U$1.SCK
- removed net SDI1: JP1.6, U$1.SDO
- removed net SDO1: JP1.7, U$1.SDI
- removed net WAKE_MRF24J40MA: JP1.4, U$1.WAKE
- new net CE: JP1.14, SV1.3
- new net CSN: JP1.13, SV1.4
- new net IRQ0: JP1.18, R1.1, SV1.8
- new net MISO: JP1.7, SV1.7
- new net MOSI: JP1.6, SV1.6
- new net RX: JP1.3
- new net SCK: JP1.5, SV1.5
- new net TX: JP1.4
- net +3V3: now also SV1.2; no longer U$1.VIN
- net GND: now also SV1.1; no longer U$1.GND1, U$1.GND2, U$1.GND3
Other:
- note added: "Kiev nrf24L01 expansion"
- note removed: "Leicester - 802.15.4 expansion"
